File: Thupp.kicad_pcb (KiCad board)
At the start: 2 copper layers, 42 parts

Commit message: two layer pcb, diodes on bottom.. row based
Parts:
- D10, D11, D12, D14, D15, D18, D2, D3, D4, D6, D7, D8: moved to B.Cu
- moved D15 11.2 mm to (114.3, 71.1)
- moved D11 11.2 mm to (96.5, 63.5)
- moved D17 10.4 mm to (131.8, 54.2), turned to 270 degrees
- moved D20 10.2 mm to (154.9, 55.9), turned to 270 degrees
- moved D13 9.87 mm to (113.8, 27.5)
- moved D19 9.79 mm to (151.3, 37.2)
- moved D9 9.67 mm to (94.7, 21.9)
- moved D16 9.63 mm to (132.4, 35.4)
- moved D3 8.25 mm to (57.1, 71.1), turned to 270 degrees
- moved D7 8.19 mm to (76.2, 68.6), turned to 270 degrees
- moved D10 7.85 mm to (94.7, 39.9), turned to 270 degrees
- moved D1 7.82 mm to (57.1, 32.1), turned to 270 degrees
- moved D5 7.73 mm to (75.7, 31.0), turned to 270 degrees
- moved D2 7.67 mm to (57.3, 51.4), turned to 270 degrees
- moved D18 7.62 mm to (132.1, 72.4)
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
Commit message: starting over for diodes on cols not rows
Parts:
- removed D1, D10, D11, D12, D13, D14, D15, D16, D17, D18, D19, D2, D20, D21, D3, D4, D5, D6, D7, D8, D9: D_Small, Diode_SMD:D_SOD-123
- removed MX1, MX10, MX11, MX13, MX14, MX15, MX16, MX17, MX18, MX19, MX2, MX21, MX3, MX5, MX6, MX7, MX9: MX-NoLED, Kailh_Choc:KailhChoc-1U
- removed MX12, MX20, MX8: MX-NoLED, Kailh_Choc:KailhChoc-1.5U
- removed MX4: MX-NoLED, Kailh_Choc:KailhChoc-1.75U
