File: _autosave-Thupp.kicad_pcb (KiCad board)
At the start: 2 copper layers, 150.1 x 113 mm, 42 parts

Commit message: test-list
Parts:
- moved MX1 2.13 mm to (45.6, 40.1)
- moved D1 2.08 mm to (47.7, 44.8)
